Commit message: add all

File: vrx_gazebo/worlds/example_course.world.xacro (robot description, xacro)
@@ -7,5 +7,8 @@
     <!--Waves-->
     <xacro:include filename="$(find wave_gazebo)/world_models/ocean_waves/model.xacro"/>
-    <xacro:ocean_waves/>
+    <xacro:ocean_waves gain="0" />
+    <!-- period="0"
+                     direction_x="0.0" direction_y="0.0"
+                     angle="0" -->
     <include>
       <uri>model://robotx_navigation_challenge</uri>
@@ -31,5 +34,5 @@
     </include>
     <xacro:include filename="$(find vrx_gazebo)/worlds/xacros/usv_wind_plugin.xacro"/>
-    <xacro:usv_wind_gazebo>
+    <xacro:usv_wind_gazebo direction="0">
       <wind_objs>
         <wind_obj>

File: vrx_gazebo/worlds/navigation_task.world.xacro (robot description, xacro)
@@ -1,3 +1,3 @@
-<?xml version="1.0" ?>
+<?xml version="1.0" encoding="UTF-8"?>
 <!-- World containing sandisland model and some course challenges -->
 <sdf version="1.6" xmlns:xacro="http://ros.org/wiki/xacro">
@@ -7,5 +7,5 @@
     <!--Waves-->
     <xacro:include filename="$(find wave_gazebo)/world_models/ocean_waves/model.xacro"/>
-    <xacro:ocean_waves/>
+    <xacro:ocean_waves  gain="0"/>
     <!--wind for the wamv-->
     <xacro:include filename="$(find vrx_gazebo)/worlds/xacros/usv_wind_plugin.xacro"/>

File: vrx_gazebo/worlds/xacros/usv_wind_plugin.xacro (robot description, xacro)
@@ -1,3 +1,3 @@
-<?xml version="1.0"?>
+<?xml version="1.0"  encoding="UTF-8"?>
 <world xmlns:xacro="http://ros.org/wiki/xacro">
   <xacro:macro name="usv_wind_gazebo"

File: wamv_gazebo/urdf/thruster_layouts/wamv_gazebo_thruster_config.xacro (robot description, xacro)
@@ -11,9 +11,12 @@
       <enableAngle>true</enableAngle>
       <!-- Optional Parameters -->
-      <mappingType>1</mappingType>
+      <mappingType>0</mappingType>
       <maxCmd>1.0</maxCmd>
       <maxForceFwd>250.0</maxForceFwd>
       <maxForceRev>-100.0</maxForceRev>
-      <maxAngle>${pi/2}</maxAngle>
+      <!-- <maxCmd>1.0</maxCmd>
+      <maxForceFwd>250.0</maxForceFwd>
+      <maxForceRev>-100.0</maxForceRev> -->
+      <maxAngle>${pi/6}</maxAngle>
     </thruster>
   </xacro:macro>

File: wamv_gazebo/urdf/wamv_gazebo.xacro (robot description, xacro)
@@ -1,3 +1,4 @@
-<?xml version="1.0"?>
+<?xml version="1.0"  encoding="UTF-8"?>
+<!-- 中文 -->
 <robot xmlns:xacro="http://ros.org/wiki/xacro">
   <!-- Macro to create a WAM-V with dyanmics plugins and a customizeable thruster layout -->

File: wamv_gazebo/urdf/ywamv_gazebo.urdf.xacro (robot description, xacro)
@@ -48,8 +48,4 @@
     <xacro:if value="${thruster_conf == 'T'}">
       <xacro:wamv_gazebo thruster_layout="$(find wamv_gazebo)/urdf/thruster_layouts/wamv_t_thrusters.xacro"/>
-    </xacro:if>
-    <!-- WAMV with "T" thruster configuration -->
-    <xacro:if value="${thruster_conf == 'O'}">
-      <xacro:wamv_gazebo thruster_layout="$(find wamv_gazebo)/urdf/thruster_layouts/wamv_one_thrusters.xacro"/>
     </xacro:if>
     <!-- WAMV with "X" thruster configuration -->

File: wave_gazebo/world_models/ocean_waves/model.xacro (robot description, xacro)
@@ -17,7 +17,10 @@
 -->
 <world xmlns:xacro="http://ros.org/wiki/xacro">
-  <xacro:macro name="ocean_waves" params="gain:=0.1 period:=5
+  <xacro:macro name="ocean_waves" params="gain:=0.0 period:=5
                      direction_x:=1.0 direction_y:=0.0
                      angle:=0.4">
+  <!-- <xacro:macro name="ocean_waves" params="gain:=0.1 period:=5
+                     direction_x:=1.0 direction_y:=0.0
+                     angle:=0.4"> -->
   <model name='ocean_waves'>
     <static>true</static>
